File: MPe_V6_WORK/MPeV6PCB/MPeV6PCB.kicad_pcb (KiCad board)
At the start: 2 copper layers, 135.2 x 59.5 mm, 73 parts, among them J1 UART, J10 TO, J2 SPI, J3 D9, J4 D4, J5 A2, J6 PAS2, J7 TIN, J8 BAT, J9 CUR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

Commit message: zmiana
Parts:
- removed R24: 10K, Resistor_SMD:R_0805_2012Metric_Pad1.20x1.40mm_HandSolder
- added R7: 2.2k, Resistor_SMD:R_0805_2012Metric_Pad1.20x1.40mm_HandSolder, F.Cu at (184.0, 98.5)
- R27: value 10K -> 1k
Connections:
- A1 pad 2: Net-(A1-D0/RX) -> RX_2
- R28 pad 2: Net-(A1-D0/RX) -> RX_2
Routing:
- net RX_2: track 64.9 -> 75.3 mm
- net Net-(A1-D0/RX): track 8.90 -> 0.00 mm
- net TX_2: track 41.3 -> 43.6 mm
- net GND: track 15.2 -> 16.0 mm, vias 100 -> 191
- net (no net): vias 0 -> 1
Other:
- outline, holes or cut-outs redrawn
